File: hardware/inputs.kicad_sch (KiCad schematic)
At the start: 8 parts, among them U4 ADA4098-2BCPZ-RL7

Commit message: finished single board layout - upping to panel size
Parts:
- removed R13, R6: 100k, PCM_SparkFun-Resistor:R_0402_1005Metric, symbol PCM_SparkFun-Resistor:100k_0402
- added R13, R6: 100k, Resistor_SMD:R_0402_1005Metric, symbol partywagon112_partdb:ERJ-2RKF1003X
Connections:
- net GND: now also R13.1, R6.1
- net IN0: now also R6.2
- net IN1: now also R13.2
